File: MS5837_mount/MS5837_mount.sch (KiCad schematic (older format))
At the start: 3 parts, among them P1 CONN_01X04, U1 MS5837-30BA

Commit message: Add pcb
Parts:
- U1: footprint (none) -> MS5837:MS5837-BA30
Changed lines of the file:
@@
 LIBS:valves
 LIBS:ms5837-30ba
+LIBS:MS5837_mount-cache
 EELAYER 25 0
 EELAYER END
@@
 F 0 "U1" H 1250 1500 60  0000 C CNN
 F 1 "MS5837-30BA" H 1300 1900 60  0000 C CNN
-F 2 "" H 1450 1900 60  0001 C CNN
+F 2 "MS5837:MS5837-BA30" H 1450 1900 60  0001 C CNN
 F 3 "" H 1450 1900 60  0000 C CNN
 	1    1400 1900

Commit message: Make pcb round
Parts:
- removed P1: CONN_01X04, Pin_Headers:Pin_Header_Straight_1x04, symbol CONN_01X04
- added P1, P2: CONN_01X02, Pin_Headers:Pin_Header_Straight_1x02, symbol CONN_01X02
Connections:
- net GND: now also P1.2 (P2)
- net VCC: now also P1.1 (P1)
- net at U1.3 (SCL): now also P2.1 (P1)
- net at U1.4 (SDA): now also P2.2 (P2)
Changed lines of the file:
@@
-$EndComp
-$Comp
-L CONN_01X04 P1
-U 1 1 588BAA97
-P 2300 2050
-F 0 "P1" H 2300 2300 50  0000 C CNN
-F 1 "CONN_01X04" V 2400 2050 50  0000 C CNN
-F 2 "Pin_Headers:Pin_Header_Straight_1x04" H 2300 2050 50  0001 C CNN
-F 3 "" H 2300 2050 50  0000 C CNN
-	1    2300 2050
-	1    0    0    -1
 $EndComp
 $Comp
@@
 L GND #PWR02
 U 1 1 588BB7B1
-P 2050 1750
-F 0 "#PWR02" H 2050 1500 50  0001 C CNN
-F 1 "GND" H 2050 1600 50  0000 C CNN
-F 2 "" H 2050 1750 50  0000 C CNN
-F 3 "" H 2050 1750 50  0000 C CNN
-	1    2050 1750
+P 1800 1500
+F 0 "#PWR02" H 1800 1250 50  0001 C CNN
+F 1 "GND" H 1800 1350 50  0000 C CNN
+F 2 "" H 1800 1500 50  0000 C CNN
+F 3 "" H 1800 1500 50  0000 C CNN
+	1    1800 1500
 	-1   0    0    1
 $EndComp
@@
 L VCC #PWR03
 U 1 1 588BB7CE
-P 1850 1750
-F 0 "#PWR03" H 1850 1600 50  0001 C CNN
-F 1 "VCC" H 1850 1900 50  0000 C CNN
-F 2 "" H 1850 1750 50  0000 C CNN
-F 3 "" H 1850 1750 50  0000 C CNN
-	1    1850 1750
+P 2000 1500
+F 0 "#PWR03" H 2000 1350 50  0001 C CNN
+F 1 "VCC" H 2000 1650 50  0000 C CNN
+F 2 "" H 2000 1500 50  0000 C CNN
+F 3 "" H 2000 1500 50  0000 C CNN
+	1    2000 1500
 	1    0    0    -1
 $EndComp
-Wire Wire Line
-	2100 2200 1800 2200
-Wire Wire Line
-	2100 2100 1800 2100
-Wire Wire Line
-	1800 2100 1800 2050
-Wire Wire Line
-	2050 1750 2050 1900
-Wire Wire Line
-	2050 1900 2100 1900
-Wire Wire Line
-	1850 1750 1850 2000
-Wire Wire Line
-	1850 2000 2100 2000
-Wire Wire Line
-	1000 2050 800  2050
-Wire Wire Line
-	1000 2200 1000 2350
-Wire Wire Line
-	1000 2350 800  2350
-Wire Wire Line
-	800  2350 800  2450
 $Comp
 L VCC #PWR04
@@
 	1    0    0    -1
 $EndComp
-Wire Wire Line
-	800  2050 800  1750
 $Comp
 L PWR_FLAG #FLG05
@@
 	1    0    0    -1
 $EndComp
+$Comp
+L CONN_01X02 P2
+U 1 1 58E3A656
+P 2300 2150
+F 0 "P2" H 2300 2300 50  0000 C CNN
+F 1 "CONN_01X02" V 2400 2150 50  0000 C CNN
+F 2 "Pin_Headers:Pin_Header_Straight_1x02" H 2300 2150 50  0001 C CNN
+F 3 "" H 2300 2150 50  0000 C CNN
+	1    2300 2150
+	1    0    0    -1
+$EndComp
+$Comp
+L CONN_01X02 P1
+U 1 1 58E3A69D
+P 2300 1600
+F 0 "P1" H 2300 1750 50  0000 C CNN
+F 1 "CONN_01X02" V 2400 1600 50  0000 C CNN
+F 2 "Pin_Headers:Pin_Header_Straight_1x02" H 2300 1600 50  0001 C CNN
+F 3 "" H 2300 1600 50  0000 C CNN
+	1    2300 1600
+	1    0    0    -1
+$EndComp
+Wire Wire Line
+	2100 2200 1800 2200
+Wire Wire Line
+	1800 2100 1800 2050
+Wire Wire Line
+	1000 2050 800  2050
+Wire Wire Line
+	1000 2200 1000 2350
+Wire Wire Line
+	1000 2350 800  2350
+Wire Wire Line
+	800  2350 800  2450
+Wire Wire Line
+	800  2050 800  1750
 Wire Wire Line
 	800  950  800  1100
 Wire Wire Line
 	1200 950  1200 1100
+Wire Wire Line
+	2100 1550 2000 1550
+Wire Wire Line
+	2000 1550 2000 1500
+Wire Wire Line
+	2100 1650 1800 1650
+Wire Wire Line
+	1800 1650 1800 1500
+Wire Wire Line
+	2100 2100 1800 2100
 $EndSCHEMATC
